Commit message: edit

File: install/mobile_robot/share/mobile_robot/model/robot.xacro (robot description, xacro)
@@ -65,5 +65,5 @@
 <!-- This macro defines the complete inertial section of the wheel -->
 <!-- It is used later in the code -->
-<xacro:macro name="inertial_wheel">
+<xacro:macro name="inertia_wheel">
     <inertial>
     <origin rpy="1.570795 0 0" xyz="0 0 0"/>
@@ -76,6 +76,6 @@
 <xacro:macro name="inertia_caster">
     <inertial>
-    <oritin rpy="0 0 0" xyz="0 0 0"/>
-    <mass value="{m3}"/>
+    <origin rpy="0 0 0" xyz="0 0 0"/>
+    <mass value="${m3}"/>
     <inertia ixx="${I_caster}" ixy="0.0" ixz="0.0" iyy="${I_caster}" iyz="0" izz="${I_caster}" />
     </inertial>
@@ -204,5 +204,5 @@
         </geometry>
     </collision>
-    <xacro:inertia_wheel />
+    <xacro:inertia_caster />
 </link>
 <!-- ###########################################################   -->

Commit message: edit

File: install/mobile_robot/share/mobile_robot/model/robot.xacro (robot description, xacro)
@@ -81,4 +81,44 @@
     </inertial>
 </xacro:macro>
+<!-- ###########################################################    -->
+<!--     Aesthetic top ball (with collision)                        -->
+<!-- ###########################################################    -->
+<!-- Ball radius -->
+<xacro:property name="r_ball" value="0.2"/>
+<!-- Ball material density (reuse d3 or make a new one) -->
+<xacro:property name="d_ball" value="${d3}"/>
+<!-- Ball mass (solid sphere) -->
+<xacro:property name="m_ball" value="${d_ball*(4.0/3.0)*pi_const*r_ball*r_ball*r_ball}"/>
+<!-- Ball inertia (solid sphere): I = 2/5 m r^2 -->
+<xacro:property name="I_ball" value="${(2.0/5.0)*m_ball*r_ball*r_ball}"/>
+<xacro:macro name="inertia_ball">
+  <inertial>
+    <origin rpy="0 0 0" xyz="0 0 0"/>
+    <mass value="${m_ball}"/>
+    <inertia ixx="${I_ball}" ixy="0.0" ixz="0.0"
+             iyy="${I_ball}" iyz="0.0"
+             izz="${I_ball}" />
+  </inertial>
+</xacro:macro>
+<!-- ###########################################################    -->
+<!--     Aesthetic Ear                     -->
+<!-- ###########################################################    -->
+<!-- Ear radius -->
+<xacro:property name="r_ear" value="0.1333"/>
+<!-- Ear material density (reuse d3 or make a new one) -->
+<xacro:property name="d_ear" value="${d3}"/>
+<!-- Ear mass (solid sphere) -->
+<xacro:property name="m_ear" value="${d_ear*(4.0/3.0)*pi_const*r_ear*r_ear*r_ear}"/>
+<!-- Ear inertia (solid sphere): I = 2/5 m r^2 -->
+<xacro:property name="I_ear" value="${(2.0/5.0)*m_ear*r_ear*r_ear}"/>
+<xacro:macro name="inertia_ear">
+  <inertial>
+    <origin rpy="0 0 0" xyz="0 0 0"/>
+    <mass value="${m_ear}"/>
+    <inertia ixx="${I_ear}" ixy="0.0" ixz="0.0"
+             iyy="${I_ear}" iyz="0.0"
+             izz="${I_ear}" />
+  </inertial>
+</xacro:macro>
 <!-- ###########################################################   -->
 <!-- ###########################################################   -->
@@ -209,3 +249,82 @@
 <!-- END: Caster wheel -->
 <!-- ###########################################################   -->
+<!-- ###########################################################   -->
+<!-- START: Ball on top of chassis (visual + collision)            -->
+<!-- ###########################################################   -->
+<joint name="top_ball_joint" type="fixed">
+  <parent link="body_link"/>
+  <child link="top_ball_link"/>
+  <!-- Top of chassis is at z = s1 + b/2, then add the ball radius -->
+  <origin xyz="0 0 ${s1 + b/2 + r_ball}" rpy="0 0 0"/>
+</joint>
+<link name="top_ball_link">
+  <visual>
+    <origin xyz="0 0 0" rpy="0 0 0"/>
+    <geometry>
+      <sphere radius="${r_ball}"/>
+    </geometry>
+  </visual>
+  <collision>
+    <origin xyz="0 0 0" rpy="0 0 0"/>
+    <geometry>
+      <sphere radius="${r_ball}"/>
+    </geometry>
+  </collision>
+  <xacro:inertia_ball />
+</link>
+<!-- ###########################################################   -->
+<!-- END: Ball on top of chassis                                   -->
+<!-- ###########################################################   -->
+<!-- ###########################################################   -->
+<!-- START: Left Ear (visual + collision)            -->
+<!-- ###########################################################   -->
+<joint name="left_ear_joint" type="fixed">
+  <parent link="top_ball_link"/>
+  <child link="left_ear_link"/>
+  <origin xyz="0 ${r_ball*0.7071 + r_ear*0.5} ${r_ball*0.7071 + r_ear*0.5}" rpy="0 0 0"/>
+</joint>
+<link name="left_ear_link">
+  <visual>
+    <origin xyz="0 0 0" rpy="0 0 0"/>
+    <geometry>
+      <sphere radius="${r_ear}"/>
+    </geometry>
+  </visual>
+  <collision>
+    <origin xyz="0 0 0" rpy="0 0 0"/>
+    <geometry>
+      <sphere radius="${r_ear}"/>
+    </geometry>
+  </collision>
+  <xacro:inertia_ear />
+</link>
+<!-- ###########################################################   -->
+<!-- END: Left Ear (visual + collision)                                   -->
+<!-- ###########################################################   -->
+<!-- ###########################################################   -->
+<!-- START: Right Ear (visual + collision)            -->
+<!-- ###########################################################   -->
+<joint name="right_ear_joint" type="fixed">
+  <parent link="top_ball_link"/>
+  <child link="right_ear_link"/>
+  <origin xyz="0 ${-r_ball*0.7071 - r_ear*0.5} ${r_ball*0.7071 + r_ear*0.5}" rpy="0 0 0"/>
+</joint>
+<link name="right_ear_link">
+  <visual>
+    <origin xyz="0 0 0" rpy="0 0 0"/>
+    <geometry>
+      <sphere radius="${r_ear}"/>
+    </geometry>
+  </visual>
+  <collision>
+    <origin xyz="0 0 0" rpy="0 0 0"/>
+    <geometry>
+      <sphere radius="${r_ear}"/>
+    </geometry>
+  </collision>
+  <xacro:inertia_ear />
+</link>
+<!-- ###########################################################   -->
+<!-- END: Right Ear (visual + collision)                                   -->
+<!-- ###########################################################   -->
 </robot>

Commit message: edit

File: install/mobile_robot/share/mobile_robot/model/robot.xacro (robot description, xacro)
@@ -328,3 +328,36 @@
 <!-- END: Right Ear (visual + collision)                                   -->
 <!-- ###########################################################   -->
+<!-- ###########################################################   -->
+<!-- START: LIDAR            -->
+<!-- ###########################################################   -->
+<joint name="lidar_joint" type="fixed">
+    <origin xyz="0.0 0 ${b+r}" rpy="0 0 0"/>
+    <parent link="body_link"/>
+    <child link="lidar_link"/>
+    <axis xyz="0 1 0" rpy="0 0 0"/>
+</joint>
+<link name='lidar_link'>
+    <visual>
+      <origin xyz="0 0 0.05" rpy="0 0 0"/>
+      <geometry>
+        <cylinder length="0.1" radius="0.1"/>
+      </geometry>
+    </visual>
+    <collision name='collision'>
+      <origin xyz="0 0 0.05" rpy="0 0 0"/>
+      <geometry>
+        <cylinder length="0.1" radius="0.1"/>
+      </geometry>
+    </collision>
+    <inertial>
+      <mass value="1e-6"/>
+      <origin xyz="0 0 0" rpy="0 0 0"/>
+      <inertia ixx="1e-6" ixy="0" ixz="0"
+               iyy="1e-6" iyz="0" izz="1e-6"
+      />
+    </inertial>
+</link>
+<!-- ###########################################################   -->
+<!-- END: LIDAR            -->
+<!-- ###########################################################   -->
 </robot>

Commit message: edit

File: install/mobile_robot/share/mobile_robot/model/robot.xacro (robot description, xacro)
@@ -252,9 +252,11 @@
 <!-- START: Ball on top of chassis (visual + collision)            -->
 <!-- ###########################################################   -->
-<joint name="top_ball_joint" type="fixed">
+<joint name="top_ball_joint" type="continuous">
   <parent link="body_link"/>
   <child link="top_ball_link"/>
-  <!-- Top of chassis is at z = s1 + b/2, then add the ball radius -->
   <origin xyz="0 0 ${s1 + b/2 + r_ball}" rpy="0 0 0"/>
+  <axis xyz="0 0 1"/>
+  <limit effort="5.0" velocity="2.0"/>
+  <dynamics damping="0.2" friction="0.0"/>
 </joint>
 <link name="top_ball_link">
